File: RBoard.sch (KiCad schematic (older format))
At the start: 4 parts

Commit message: Updated firmware. Added schematic PDF.
Other:
- note added: "1"
- note added: "2"
- note added: "3"
- note added: "4"
- note added: "Connectors"
- note added: "Little Brain"
- note added: "Microcontroller"
- note added: "Power"
- note added: "Sensors"
- moved on the sheet: H1, H2, H3, H4
Changed lines of the file:
@@
 $EndDescr
 $Sheet
-S 1500 1500 1000 1000
+S 2750 2250 1000 1000
 U 5F83BB42
 F0 "Power" 50
@@
 $EndSheet
 $Sheet
-S 3000 1500 1000 1000
+S 5250 2250 1000 1000
 U 5F83BC83
 F0 "Microcontroller" 50
@@
 $EndSheet
 $Sheet
-S 1500 3000 1000 1000
+S 2750 4750 1000 1000
 U 5F83C004
 F0 "Sensors" 50
@@
 $EndSheet
 $Sheet
-S 3000 3000 1000 1000
+S 5250 4750 1000 1000
 U 5F83C1A4
 F0 "Connectors" 50
@@
 L Mechanical:MountingHole H1
 U 1 1 5FB1AA99
-P 6250 1500
-F 0 "H1" H 6350 1546 50  0000 L CNN
-F 1 "MountingHole" H 6350 1455 50  0000 L CNN
-F 2 "MountingHole:MountingHole_3.2mm_M3" H 6250 1500 50  0001 C CNN
-F 3 "~" H 6250 1500 50  0001 C CNN
-	1    6250 1500
+P 7650 2375
+F 0 "H1" H 7750 2421 50  0000 L CNN
+F 1 "MountingHole" H 7750 2330 50  0000 L CNN
+F 2 "MountingHole:MountingHole_3.2mm_M3" H 7650 2375 50  0001 C CNN
+F 3 "~" H 7650 2375 50  0001 C CNN
+	1    7650 2375
 	1    0    0    -1
 $EndComp
@@
 L Mechanical:MountingHole H2
 U 1 1 5FB1AE5C
-P 6250 1750
-F 0 "H2" H 6350 1796 50  0000 L CNN
-F 1 "MountingHole" H 6350 1705 50  0000 L CNN
-F 2 "MountingHole:MountingHole_3.2mm_M3" H 6250 1750 50  0001 C CNN
-F 3 "~" H 6250 1750 50  0001 C CNN
-	1    6250 1750
+P 7650 2625
+F 0 "H2" H 7750 2671 50  0000 L CNN
+F 1 "MountingHole" H 7750 2580 50  0000 L CNN
+F 2 "MountingHole:MountingHole_3.2mm_M3" H 7650 2625 50  0001 C CNN
+F 3 "~" H 7650 2625 50  0001 C CNN
+	1    7650 2625
 	1    0    0    -1
 $EndComp
@@
 L Mechanical:MountingHole H3
 U 1 1 5FB1B3B8
-P 6250 2000
-F 0 "H3" H 6350 2046 50  0000 L CNN
-F 1 "MountingHole" H 6350 1955 50  0000 L CNN
-F 2 "MountingHole:MountingHole_3.2mm_M3" H 6250 2000 50  0001 C CNN
-F 3 "~" H 6250 2000 50  0001 C CNN
-	1    6250 2000
+P 7650 2875
+F 0 "H3" H 7750 2921 50  0000 L CNN
+F 1 "MountingHole" H 7750 2830 50  0000 L CNN
+F 2 "MountingHole:MountingHole_3.2mm_M3" H 7650 2875 50  0001 C CNN
+F 3 "~" H 7650 2875 50  0001 C CNN
+	1    7650 2875
 	1    0    0    -1
 $EndComp
@@
 L Mechanical:MountingHole H4
 U 1 1 5FB1B9E2
-P 6250 2250
-F 0 "H4" H 6350 2296 50  0000 L CNN
-F 1 "MountingHole" H 6350 2205 50  0000 L CNN
-F 2 "MountingHole:MountingHole_3.2mm_M3" H 6250 2250 50  0001 C CNN
-F 3 "~" H 6250 2250 50  0001 C CNN
-	1    6250 2250
+P 7650 3125
+F 0 "H4" H 7750 3171 50  0000 L CNN
+F 1 "MountingHole" H 7750 3080 50  0000 L CNN
+F 2 "MountingHole:MountingHole_3.2mm_M3" H 7650 3125 50  0001 C CNN
+F 3 "~" H 7650 3125 50  0001 C CNN
+	1    7650 3125
 	1    0    0    -1
 $EndComp
+Wire Notes Line
+	7500 3250 8300 3250
+Wire Notes Line
+	8300 3250 8300 2250
+Wire Notes Line
+	8300 2250 7500 2250
+Wire Notes Line
+	7500 2250 7500 3250
+Text Notes 675  1250 0    295  ~ 59
+Little Brain
+Text Notes 3075 2925 0    295  ~ 59
+1
+Text Notes 5575 2925 0    295  ~ 59
+2
+Text Notes 3075 5450 0    295  ~ 59
+3
+Text Notes 5550 5475 0    295  ~ 59
+4
+Text Notes 2725 2125 0    98   ~ 20
+Power
+Text Notes 5225 2125 0    98   ~ 20
+Microcontroller
+Text Notes 2725 4625 0    98   ~ 20
+Sensors
+Text Notes 5225 4625 0    98   ~ 20
+Connectors
 $EndSCHEMATC
